Commit message: Edit catkin_ws in V3.5 for First Video Version

File: ROS_V3/ROS V3.5/catkin_ws/src/car_test/urdf/car.xacro (robot description, xacro)
@@ -21,5 +21,5 @@
 <xacro:property name="wheel_width" value="0.2"/>
 <xacro:property name="wheel_height" value="0.8"/>
-<xacro:property name="wheel_mass" value="30"/>
+<xacro:property name="wheel_mass" value="1"/>
 <!-- /////////////////////////////////////////////////////-->
 <xacro:macro name="cylinder_inertia" params ="m r h">
@@ -68,5 +68,5 @@
       </geometry>
     </collision>
-   <xacro:inertial_matrix mass="5"/>
+   <xacro:inertial_matrix mass="1"/>
  </link>
  <gazebo reference="chassis">
@@ -89,8 +89,8 @@
   </link>
 <gazebo reference ="${prefix}_${suffix}_w">
-    <mu1 value="200.0"/>
-    <mu2 value="100.0"/>
-    <kp value="10000000.0"/>
-    <kd value= "1.0"/>
+    <mu1 value="1000000.0"/>
+    <mu2 value="1000000.0"/>
+    <kp value="1000000.0"/>
+    <kd value= "1000000.0"/>
     <material>Gazebo/Black</material>
 </gazebo>
@@ -100,5 +100,5 @@
   <origin xyz= "${X} ${Y} ${Z}" rpy="0 0 0"/>
   <axis xyz="0 1 0"/>
-  <limit effort= "100" velocity="100"/>
+  <limit effort= "5" velocity="10000"/>
   <dynamics damping="0.0" friction="0.0"/>
 </joint>
