Commit message: Edit README

File: ROS_V3/ROS V3.4/catkin_ws/src/car_test/urdf/car.xacro (robot description, xacro)
@@ -21,6 +21,7 @@
 <xacro:property name="wheel_width" value="0.2"/>
 <xacro:property name="wheel_height" value="0.8"/>
-<xacro:property name="wheel_mass" value="10"/>
+<xacro:property name="wheel_mass" value="1"/>
 <!-- /////////////////////////////////////////////////////-->
+<!-- Macro for computing cylinder inertia, useful for dynamic simulations -->
 <xacro:macro name="cylinder_inertia" params ="m r h">
   <inertial>
@@ -32,4 +33,5 @@
 </xacro:macro>
 <!-- ///////////////////////////////////////////////////-->
+<!-- Macro to provide a simple inertial matrix for parts -->
 <xacro:macro name= "inertial_matrix" params="mass">
   <inertial>
@@ -68,5 +70,5 @@
       </geometry>
     </collision>
-   <xacro:inertial_matrix mass="5"/>
+   <xacro:inertial_matrix mass="1"/>
  </link>
  <gazebo reference="chassis">
@@ -74,5 +76,6 @@
     <material>Gazebo/Red</material>
   </gazebo>
-<!-- ///////////////////      Wheels      ///////////////////////   -->
+<!-- //////////////////////////////////////////   -->
+<!-- wheels-->
 <xacro:macro name="wheel" params= "prefix suffix X Y Z">
   <link name= "${prefix}_${suffix}_w">
@@ -88,4 +91,5 @@
   <xacro:cylinder_inertia m="${wheel_mass}" r="${wheel_radius}" h="${wheel_width}"/>
   </link>
+<!-- friction parameters-->
 <gazebo reference ="${prefix}_${suffix}_w">
     <mu1 value="1000000.0"/>
@@ -100,5 +104,5 @@
   <origin xyz= "${X} ${Y} ${Z}" rpy="0 0 0"/>
   <axis xyz="0 1 0"/>
-  <limit effort= "10000" velocity="10000"/>
+  <limit effort= "5" velocity="10000"/>
   <dynamics damping="0.0" friction="0.0"/>
 </joint>
